Commit message: tried to change shape of link to cylinder, unsuccessful

File: urdf/robot.urdf (robot description, URDF)
Before this commit: robot robot, 2 links, 1 joints
Links:
- link link_chassis: geometry collision cylinder length=25 radius=30; visual cylinder length=25 radius=30

Commit message: cylinder is worked out... need to figure out the math on the links and joints... not clicking yet... need more time

File: urdf/robot.urdf (robot description, URDF)
Before this commit: robot robot, 2 links, 1 joints
Links:
- link link_chassis: geometry collision cylinder length=.30 radius=.25; visual cylinder length=.30 radius=.25
Joints:
- joint joint_chassis_left_wheel: origin xyz=-0.5 0.65 0 rpy=0 0 0 -> xyz=-0.25 0.65 0 rpy=0 0 0

Commit message: continue onto mesh after you have built up the base for building robots.

File: urdf/robot.urdf (robot description, URDF)
Before this commit: robot robot, 2 links, 1 joints
Links:
- added link link_caster_wheel, mass 1; collision sphere radius=0.10; collision sphere radius=0.2
- added link link_right_wheel, mass 1; collision cylinder length=0.12 radius=0.08; collision cylinder length=0.12 radius=0.4
- link link_chassis: geometry collision box size=2 1.3 0.4; visual box size=2 1.3 0.4
- link link_left_wheel: geometry collision cylinder length=0.12 radius=0.08; collision cylinder length=0.12 radius=0.4
Joints:
- added joint joint_chassis_caster_wheel: type fixed, parent link_chassis, child link_caster_wheel, origin xyz=0.8 0 -0.15 rpy=0 0 0
- added joint joint_chassis_right_wheel: type continuous, parent link_chassis, child link_right_wheel, origin xyz=-0.5 -0.65 0 rpy=0 0 0, axis 0 1 0, limit effort=10000 velocity=1000
- joint joint_chassis_left_wheel: origin xyz=-0.25 0.65 0 rpy=0 0 0 -> xyz=-0.5 0.65 0 rpy=0 0 0
